File: MSMGDustSensor/MSMGDustSensor.sch (EAGLE design)
At the start: 0 parts

Commit message: schematic almost done
Parts:
- added C1, C2, C3: 0.1uF, MSMG:C0603(1608)
- added D1, D2: MBR120, MSMG:MBR120
- added J1: POWER_JACK, MSMG:POWER_JACK
- added JP1: PARTICLE_PHOTON, MSMG:PARTICLE_PHOTON
- added LED1, LED2: LFH1056, MSMG:LFH1056
- added LED3: (no value), MSMG:LED3MM
- added Q1: BC817-16LT1SMD, MSMG:BC817-16LT1SMD
- added R1, R2, R3, R4, R5, R6: (no value), MSMG:R0603(1608)
- added R10, R9: 470, MSMG:R0603(1608)
- added R11, R12, R14, R15, R16, R18: 4.7k, MSMG:R0603(1608)
- added R13, R7, R8: 1k, MSMG:R0603(1608)
- added R17: 47k, MSMG:R0603(1608)
- added S1: (no value), WaterDrop:SWITCH
- added TR1, TR2, TR3: DMN2041L, MSMG:DMN2041L
- added U1: HPMA115S0-XXX, MSMG:HPMA115S0-XXX
- added U2: BUZZER, MSMG:BUZZER
- added U3: BME280, MSMG:BME280
- added U4: MCP6002-SO8, MSMG:MCP6002-SO8
- added X1: 53261-0871, MSMG:53261-0871
Connections:
- new net 3.3V: C2.1, JP1.+3V3, R11.2, R12.2, U3.VIN, U4G$3.V+
- new net 5V: C1.1, D1.C, D2.C, JP1.VIN, R1.2, R13.1, R2.2, R3.2, R8.1, S1.P$1, U2.P$1, X1.2
- new net A0: JP1.A0, U4B.-IN, U4B.OUT
- new net A1: JP1.A1, U4A.-IN, U4A.OUT
- new net BLUE_LED: JP1.(JTAG_TMS)D7, R4.2, TR1.G
- new net BUZZER_PWM: JP1.(JTAG_TRST)D3, R7.2
- new net GND: C1.2, C2.2, C3.2, J1.GND, J1.GNDBREAK, JP1.GND@2, JP1.GND@21, LED3.C, Q1.E, R15.2, R17.2, R4.1, R5.1, R6.1, TR1.S, TR2.S, TR3.S, U3.GND, U4G$3.V-, X1.8
- new net GREEN_LED: JP1.(JTAG_TCK)D6, R5.2, TR2.G
- new net N$1: D1.A, J1.PWR
- new net N$11: R17.1, R18.2, S1.P$2
- new net N$13: Q1.C, R8.2, U2.P$2
- new net N$14: C3.1, R15.1, R16.2, U4B.+IN
- new net N$15: LED1.R+, LED2.R+, R3.1
- new net N$16: U4A.+IN
- new net N$17: LED3.A, R13.2
- new net N$18: Q1.B, R7.1
- new net N$2: D2.A
- new net N$3: LED1.B+, LED2.B+, R1.1
- new net N$4: LED1.G+, LED2.G+, R2.1
- new net N$5: JP1.TX, R9.1
- new net N$6: LED1.B-, LED2.B-, TR1.D
- new net N$7: LED1.G-, LED2.G-, TR2.D
- new net N$8: LED1.R-, LED2.R-, TR3.D
- new net N$9: JP1.RX, R10.1
- new net RED_LED: JP1.(JTAG_TDI)D5, R6.2, TR3.G
- new net RXD: R10.2, X1.6
- new net SCL: JP1.(SCL)D1, R12.1, U3.SCK
- new net SDA: JP1.(SDA)D0, R11.1, U3.SDI
- new net TEST: JP1.(JTAG_TDO)D4, R18.1
- new net TXD: R9.2, X1.7
- new net VBAT: R16.1
Other:
- note added: "battery + dc/dc board ext pins"

Commit message: schematic almost done
Parts:
- added C4, C5, C6: 0.1uF, MSMG:C0603(1608)
- added J2: (no value), SparkFun-Connectors:CONN_04
- added U5: TSL2591, MSMG:TSL2591
- added U6: BME280, MSMG:BME280
- R15, R16: value 4.7k -> 47k
- U3: value BME280 -> BME280BOARD; device MSMG:BME280 -> MSMG:BME280BOARD
Connections:
- net 3.3V: now also C4.1, C5.1, C6.1, J2.1, S1.P$1, U5.VDD, U6.VDD, U6.VDDIO
- net 5V: no longer S1.P$1
- net GND: now also C4.2, C5.2, C6.2, J2.4, U5.GND, U6.GND@1, U6.GND@7
- net SCL: now also J2.2, U5.SCL, U6.SCK
- net SDA: now also J2.3, U5.SDA, U6.SDI
Other:
- moved on the sheet: C1, C2, C3, D1, D2, J1, JP1, LED1, LED2, LED3, Q1, R1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

Commit message: schematic clean up
Parts:
- added J3: (no value), SparkFun-Connectors:CONN_04
Connections:
- net 5V: now also J3.1
- net GND: now also J3.4
- net N$2: now also J3.3
- net VBAT: now also J3.2
Other:
- moved on the sheet: C1, C2, C3, C4, C5, C6, D1, D2, J1, J2, JP1, LED1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

Commit message: board file almost done
Parts:
- removed U5: TSL2591, MSMG:TSL2591
- added C7: 0.1uF, MSMG:C0603(1608)
- added H1, H2, H3, H4: MOUNT-PAD-ROUND3.2, holes:MOUNT-PAD-ROUND3.2
- added J4, J5, J6: (no value), SparkFun-Connectors:CONN_04
- added JP2: PARTICLE_PHOTON, MSMG:PARTICLE_PHOTON
- added R19: 1k, MSMG:R0603(1608)
- added X2: 5268-02, OSSI:5268-02
- J1: value POWER_JACK -> (none); device MSMG:POWER_JACK -> SparkFun-Connectors:CONN_03
- J2: value (none) -> POWER_JACK; device SparkFun-Connectors:CONN_04 -> MSMG:POWER_JACK
- JP1: value PARTICLE_PHOTON -> JP2; device MSMG:PARTICLE_PHOTON -> GFE:JP2
- LED1: value LFH1056 -> (none); device MSMG:LFH1056 -> MSMG:LED3MM
- LED3: value (none) -> LFH1056; device MSMG:LED3MM -> MSMG:LFH1056
- R1, R2: value (none) -> 4.7k
- R10, R9: value 470 -> 4.7k
- R11: value 4.7k -> 47k
- R12, R14, R18: value 4.7k -> (none)
- R13: value 1k -> (none)
- R15, R16: value 47k -> (none)
- R17: value 47k -> 1k
- R3, R4: value (none) -> 47k
- R5: value (none) -> 1k
- R6: value (none) -> 470
- R7: value 1k -> 470
- R8: value 1k -> 4.7k
- U1: value HPMA115S0-XXX -> MCP6002-SO8; device MSMG:HPMA115S0-XXX -> MSMG:MCP6002-SO8
- U2: value BUZZER -> TSL2591; device MSMG:BUZZER -> MSMG:TSL2591
- U4: value MCP6002-SO8 -> BME280; device MSMG:MCP6002-SO8 -> MSMG:BME280
- U6: value BME280 -> BUZZER; device MSMG:BME280 -> MSMG:BUZZER
Connections:
- removed net N$3: LED1.B+, LED2.B+, R1.1
- removed net N$6: LED1.B-, LED2.B-, TR1.D
- removed net N$8: LED1.R-, LED2.R-, TR3.D
- new net B-: J5.2, J6.2, LED2.B-, LED3.B-, R14.2
- new net G-: J5.3, J6.3, LED2.G-, LED3.G-, R16.2
- new net N$10: R14.1, TR1.D
- new net N$12: R16.1, TR2.D
- new net R-: J5.4, J6.4, LED2.R-, LED3.R-, R18.2
- net 3.3V: now also C3.1, J4.1, JP1.3, JP2.+3V3, R8.2, R9.2, U1G$3.V+, U2.VDD, U4.VDD, U4.VDDIO; no longer C2.1, J2.1, JP1.+3V3, R11.2, R12.2, U4G$3.V+, U5.VDD, U6.VDD, U6.VDDIO
- net 5V: now also C7.1, J5.1, J6.1, JP1.1, JP2.VIN, LED2.B+, LED2.G+, LED2.R+, LED3.B+, LED3.G+, LED3.R+, R19.1, R5.1, U6.P$1; no longer C1.1, JP1.VIN, R1.2, R13.1, R2.2, R3.2, R8.1, U2.P$1
- net A0: now also JP2.A0, U1B.-IN, U1B.OUT; no longer JP1.A0, U4B.-IN, U4B.OUT
- net A1: now also JP2.A1, U1A.-IN, U1A.OUT; no longer JP1.A1, U4A.-IN, U4A.OUT
- net BLUE_LED: now also JP2.(JTAG_TDI)D5, R12.2; no longer JP1.(JTAG_TMS)D7, R4.2
- net BUZZER_PWM: now also JP2.(JTAG_TRST)D3, R17.2; no longer JP1.(JTAG_TRST)D3, R7.2
- net GND: now also C7.2, J1.3, J2.GND, J2.GNDBREAK, J4.4, JP2.GND@2, JP2.GND@21, LED1.C, R11.2, R12.1, R13.1, R15.1, R2.2, R4.2, U1G$3.V-, U2.GND, U4.GND@1, U4.GND@7, X2.2; no longer J1.GND, J1.GNDBREAK, J2.4, JP1.GND@2, JP1.GND@21, LED3.C, R15.2, R17.2, R4.1, R5.1, R6.1, U4G$3.V-, U5.GND, U6.GND@1, U6.GND@7
- net GREEN_LED: now also JP2.(JTAG_TCK)D6, R13.2; no longer JP1.(JTAG_TCK)D6, R5.2
- net N$1: now also J2.PWR, X2.1; no longer J1.PWR
- net N$11: now also R10.2, R11.1; no longer R17.1, R18.2
- net N$13: now also R19.2, U6.P$2; no longer R8.2, U2.P$2
- net N$14: now also C2.1, R3.2, R4.1, U1B.+IN; no longer C3.1, R15.1, R16.2, U4B.+IN
- net N$15: now also R18.1, TR3.D; no longer LED1.R+, LED2.R+, R3.1
- net N$16: now also C1.1, R1.2, R2.1, U1A.+IN; no longer U4A.+IN
- net N$17: now also LED1.A, R5.2; no longer LED3.A, R13.2
- net N$18: now also R17.1; no longer R7.1
- net N$4: now also J1.2, R1.1; no longer LED1.G+, LED2.G+, R2.1
- net N$5: now also JP2.TX, R6.1; no longer JP1.TX, R9.1
- net N$7: now also J1.1, JP1.2; no longer LED1.G-, LED2.G-, TR2.D
- net N$9: now also JP2.RX, R7.1; no longer JP1.RX, R10.1
- net RED_LED: now also JP2.(JTAG_TMS)D7, R15.2; no longer JP1.(JTAG_TDI)D5, R6.2
- net RXD: now also R7.2; no longer R10.2
- net SCL: now also J4.2, JP2.(SCL)D1, R9.1, U2.SCL, U4.SCK; no longer J2.2, JP1.(SCL)D1, R12.1, U5.SCL, U6.SCK
- net SDA: now also J4.3, JP2.(SDA)D0, R8.1, U2.SDA, U4.SDI; no longer J2.3, JP1.(SDA)D0, R11.1, U5.SDA, U6.SDI
- net TEST: now also JP2.(JTAG_TDO)D4, R10.1; no longer JP1.(JTAG_TDO)D4, R18.1
- net TXD: now also R6.2; no longer R9.2
- net VBAT: now also R3.1; no longer R16.1
Other:
- moved on the sheet: C1, C2, C3, LED2, R1, R10, R11, R12, R13, R14, R15, R16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

Commit message: almost done
Parts:
- added U$1: MSMG_TEXT, MSMG:MSMG_TEXT
Changed lines of the file:
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@@
 <part name="X2" library="OSSI" deviceset="5268-02" device=""/>
 <part name="GND28" library="MSMG" deviceset="GND" device=""/>
+<part name="U$1" library="MSMG" deviceset="MSMG_TEXT" device=""/>
 </parts>
 <sheets>
@@
 <instance part="X2" gate="G$1" x="27.94" y="246.38" rot="R180"/>
 <instance part="GND28" gate="1" x="35.56" y="238.76"/>
+<instance part="U$1" gate="G$1" x="233.68" y="58.42"/>
 </instances>
 <busses>

Commit message: TODO added
Other:
- note added: "TODO: Connect Pin 5 to 0 for 0x76, 3.3v for 0x77 i2c address"
Changed lines of the file:
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@@
 <?xml version="1.0" encoding="utf-8"?>
 <!DOCTYPE eagle SYSTEM "eagle.dtd">
-<eagle version="8.3.0">
+<eagle version="8.3.1">
 <drawing>
 <settings>
@@
 <plain>
 <text x="43.18" y="193.04" size="1.778" layer="91">battery + dc/dc board ext pins</text>
+<text x="129.54" y="172.72" size="1.778" layer="91">TODO: Connect Pin 5 to 0 for 0x76, 3.3v for 0x77 i2c address</text>
 </plain>
 <instances>
